File: kicad/guitar.sch (KiCad schematic (older format))
At the start: 33 parts

Commit message: kicad: Some more work on the fret schematics
Parts:
- removed C? (x5): 100nF, symbol C
- removed LED? (x5): WS2812, symbol WS2812
- removed R? (x5): 47k, symbol R
- added C? (x5): 100nF, symbol C
- added LED? (x5): WS2812, symbol WS2812
- added R? (x5): 47k, symbol R
- TP: Comment Chromebook Pixel TP Connector -> Link TP Connector
Connections:
- net labels added: BUTTON, LED6
- net labels removed: ???
- wire segments 112 -> 140
Other:
- moved on the sheet: C?, R?

Commit message: kicad: Annotated components
Parts:
- removed P?: CONN_01X06, symbol CONN_01X06
- added J1: +5V, symbol CONN_01X01
- added J2: GNDPWR, symbol CONN_01X01
- added J3: +3.3V, symbol CONN_01X01
- added J4, J9: GND, symbol CONN_01X01
- added J5: SDA, symbol CONN_01X01
- added J6: SCL, symbol CONN_01X01
- added J7: TEST, symbol CONN_01X01
- added J8: ~RST, symbol CONN_01X01
- R2: renamed from R?; value 3.7k -> 4.7k
- gave numbers to parts that had none: 30
- renumbered TP to J10
Connections:
- net +3V3: now also R1.2, J3.1 (P1); no longer R1.1
- net +5V: now also J1.1 (P1)
- net GND: now also J4.1 (P1), J9.1 (P1)
- net GNDPWR: now also J2.1 (P1)
- net SCL: now also J6.1 (P1)
- net SDA: now also J5.1 (P1)
- net TEST: now also J7.1 (P1)
- net ~RST: now also R1.1, J8.1 (P1); no longer R1.2
Other:
- moved on the sheet: C8, R1
